File: board/board.kicad_pcb (KiCad board)
At the start: 2 copper layers, 21 x 13 mm, 1 part

Commit message: initial
Parts:
- added C10: 10uF, Capacitor_SMD:C_1206_3216Metric, F.Cu at (152.8, 97.3)
- added C16: 10uF, Capacitor_SMD:C_1206_3216Metric, F.Cu at (175.5, 92.7)
- added D3: SS34, Diode_SMD:D_SMA, F.Cu at (176.0, 98.8)
- added J1: 022_battery_cells, on_edge:on_edge_2x05_host, F.Cu at (185.0, 96.5)
- added J2: 000_3.3v_5v, on_edge:on_edge_2x05_device, F.Cu at (140.0, 96.5)
- added L1: 10uH, Inductor_SMD:L_Wuerth_HCI-1040, F.Cu at (168.8, 96.2)
- added Q5: HXY3404M, Package_TO_SOT_SMD:SOT-23, F.Cu at (161.3, 101.2)
- added R12: 80mR, Resistor_SMD:R_2512_6332Metric, F.Cu at (159.5, 92.0)
- added U5: CN3302, Package_SO:SOIC-8_3.9x4.9mm_P1.27mm, F.Cu at (159.5, 96.7)
- moved LOGO1 5.88 mm to (148.8, 93.2)
Routing:
- net GND: track 0.00 -> 56.6 mm, vias 0 -> 119
- net /implementation/BATT: track 0.00 -> 30.2 mm, vias 0 -> 4
- net /implementation/CE: track 0.00 -> 29.5 mm, vias 0 -> 1
- net Net-(D3-A): track 0.00 -> 14.4 mm
- net Net-(U5-CSN): track 0.00 -> 9.39 mm
- net Net-(Q5-G): track 0.00 -> 2.31 mm
- added copper zone on B.Cu, net GND
- added copper zone on F.Cu, net GND
Other:
- board size 21 x 13 mm -> 45 x 13 mm
- board text added: "osf.000"
- board text added: "osf.b167.v1.0"
